Commit message: Added launcher that visualizes icub urdf Added file for rViz and icub urdf visualization

File: icub_description/urdf/iCub.urdf (robot description, URDF)
Before this commit: robot ICub, 94 links, 93 joints
Links:
- link l6: geometry visual mesh filename=package://icub_description/meshes/l6_.dae
